File: hardware/desktopia.kicad_pcb (KiCad board)
At the start: 4 copper layers, 59.1 x 49.1 mm, 76 parts, among them J2 Prog_Connector, J3 USB4105GFA, J4 PowerMotor, J5 MotorCommandCon, U1 TPS5430DDA, U2 TCA9554DB, U3 ATmega32U4-A, U4 XC6206P182MR, U5 TXS0104EPW, U6 VL53L1CBV0FY_1, U7 CC6905S8-5FB005, Y1 X322516MLB4SI

Commit message: finish pcb
Parts:
- U4: value XC6206P182MR -> XC6206P282MR
- moved H1 3.69 mm to (101.5, 117.1)
- moved TP1 3.05 mm to (110.2, 101.9)
- moved C20 3.02 mm to (102.3, 104.4)
- moved C21 3.02 mm to (104.2, 108.7)
- moved C22 3.02 mm to (105.4, 108.7)
- moved U7 3.02 mm to (99.2, 107.6)
- moved L1 3.02 mm to (122.5, 107.5)
- moved C1 3.02 mm to (118.0, 109.1)
- moved C4 3.02 mm to (125.3, 101.4)
- moved JP1 3.02 mm to (127.8, 108.2)
- moved LED1 3.02 mm to (129.5, 105.2)
- moved R2 3.02 mm to (127.3, 104.9)
- moved D1 3.02 mm to (113.2, 109.5)
- moved R1 3.02 mm to (127.3, 106.2)
- moved R21 3.02 mm to (104.9, 106.9)
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Connections:
- net +1V8 renamed +2V8
Routing:
- net GND: track 0.00 -> 17.7 mm, vias 0 -> 55
- net +24V: track 23.5 -> 26.3 mm, vias 10 -> 18
- net /Imotor: track 20.1 -> 17.3 mm
- net +5V: track 151.2 -> 149.3 mm
- net /DC_MBside: track 41.9 -> 43.2 mm
- net /RST_MBside: track 38.9 -> 39.4 mm
- net Net-(J4-Pad1): vias 5 -> 10
- added copper zone on B.Cu, net GND
- added copper zone on F.Cu, net GND
Other:
- copper layers 4 -> 2
- board text added: "+24V"
- board text added: "+24V motor"
- board text added: "Desktopia - Motherboard"
- board text added: "GND"
- board text added: "HMI connector"
- board text added: "M_DIR"
- board text added: "M_PWM"
