File: hardware/desktopia.kicad_sch (KiCad schematic)
At the start: 0 parts

Commit message: schematic done, PCB first wip
Parts:
- added C1: 10nF, Capacitor_SMD:C_0402_1005Metric, symbol Device:C_Small
- added C10, C12, C17, C18, C19, C20, C6, C7: 100nF, Capacitor_SMD:C_0402_1005Metric, symbol Device:C_Small
- added C11, C13, C14, C15: 1uF, Capacitor_SMD:C_0402_1005Metric, symbol Device:C_Small
- added C16: 4.7uF, Capacitor_SMD:C_0402_1005Metric, symbol Device:C_Small
- added C2: 4.7uF, JLCImport:RVT1H4R7M0405_C18221489, symbol JLCImport:RVT1H4R7M0405_C18221489
- added C21: 1nF, Capacitor_SMD:C_0402_1005Metric, symbol Device:C_Small
- added C22: 100pF, Capacitor_SMD:C_0402_1005Metric, symbol Device:C_Small
- added C4: 33uF, JLCImport:VE-330M1A0505-TRO, symbol JLCImport:VE-330M1A0505-TRO
- added C8, C9: 10pF, Capacitor_SMD:C_0402_1005Metric, symbol Device:C_Small
- added D1: SS14, Diode_SMD:D_SMA, symbol Diode:SS14
- added DC1: DC050-2_5-T, JLCImport:DC050-2_5-T, symbol JLCImport:DC050-2_5-T
- added FPC_HMI1, FPC_MB1: F2D12U-A1G1-ER, JLCImport:F2D12U-A1G1-ER, symbol JLCImport:F2D12U-A1G1-ER
- added H1, H2: MountingHole_Pad, MountingHole:MountingHole_2.2mm_M2_Pad, symbol Mechanical:MountingHole_Pad
- added J1: LCD_Connector, JLCImport:LCD_round_screen, symbol Connector:Conn_01x07_Pin
- added J2: Prog_Connector, Connector_IDC:IDC-Header_2x03_P2.54mm_Vertical, symbol Connector:Conn_01x06_Pin
- added J3: USB4105GFA, JLCImport:GCT_USB4105GFA, symbol USB4105GFA:USB4105GFA
- added J4: PowerMotor, JLCImport:C508128L-2P0G36, symbol JLCImport:C508128L-2P0G36
- added J5: MotorCommandCon, JLCImport:ZX-DG28L-2_54-3P, symbol JLCImport:ZX-DG28L-2_54-3P
- added JP1: SolderJumper_2_Open, Jumper:SolderJumper-2_P1.3mm_Open_TrianglePad1.0x1.5mm, symbol Jumper:SolderJumper_2_Open
- added L1: 84uH, JLCImport:L5.8, symbol Device:L
- added LED1: KT-0603R, JLCImport:KT-0603R, symbol JLCImport:KT-0603R
- added R1, R2, R21: 100, Resistor_SMD:R_0402_1005Metric, symbol Device:R
- added R10, R11, R12, R13, R14, R19, R20, R3, R5: 10k, Resistor_SMD:R_0402_1005Metric, symbol Device:R
- added R15, R16: 5.1k, Resistor_SMD:R_0402_1005Metric, symbol Device:R
- added R17, R18, R4, R6, R7: 3.3k, Resistor_SMD:R_0402_1005Metric, symbol Device:R
- added R8, R9: 22, Resistor_SMD:R_0402_1005Metric, symbol Device:R
- added RST1: SW_Push, JLCImport:DTS41, symbol Switch:SW_Push
- added SW1, SW2, SW3, SW4, SW5: SW_Push, JLCImport:PG1350, symbol Switch:SW_Push
- added TP1, TP10, TP11, TP12, TP13, TP14, TP15, TP16, TP17, TP18, TP19, TP2, TP3, TP4, TP5, TP6, TP7, TP8, TP9: TestPoint, TestPoint:TestPoint_Pad_D1.0mm, symbol Connector:TestPoint
- added U1: TPS5430DDA, Package_SO:TI_SO-PowerPAD-8_ThermalVias, symbol Regulator_Switching:TPS5430DDA
- added U2: TCA9554DB, Package_SO:SSOP-16_5.3x6.2mm_P0.65mm, symbol Interface_Expansion:TCA9554DB
- added U3: ATmega32U4-A, Package_QFP:TQFP-44_10x10mm_P0.8mm, symbol MCU_Microchip_ATmega:ATmega32U4-A
- added U4: XC6206P182MR, Package_TO_SOT_SMD:SOT-23-3, symbol JLCImport:XC6206P182MR_C51886219
- added U5: TXS0104EPW, Package_SO:TSSOP-14_4.4x5mm_P0.65mm, symbol Logic_LevelTranslator:TXS0104EPW
- added U6: VL53L1CBV0FY_1, JLCImport:VL53L1CBV0FY_1, symbol JLCImport:VL53L1CBV0FY_1
- added U7: CC6905S8-5FB005, Package_SO:SOP-8_3.76x4.96mm_P1.27mm, symbol JLCImport:CC6905S8-5FB005
- added Y1: X322516MLB4SI, Crystal:Crystal_SMD_3225-4Pin_3.2x2.5mm, symbol Device:Crystal_GND23_Small
Connections:
- new net: R17.2, TP15.1, U5.2 (A1), U6.10 (SCL)
- new net: R19.2, TP18.1, U6.5 (XSHUT)
- new net: C12.2, U3.42 (AREF)
- new net: R3.2, R4.1, U1.4 (VSENSE)
- new net: R18.2, TP16.1, U5.3 (A2), U6.9 (SDA)
- new net: R20.2, TP17.1, U5.4 (A3), U6.7 (GPIO1)
- new net: JP1.2 (B), R1.1
- new net: R1.2, R2.1
- new net: J3.A6 (DP1), J3.B6 (DP2), R8.1
- new net: J3.A7 (DN1), J3.B7 (DN2), R9.1
- new net: J4.1, U7.3 (IP-), U7.4 (IP-)
- new net: C21.2, U7.6 (VREF)
- new net: R21.1, U7.7 (VOUT)
- new net: C1.1, D1.1 (K), L1.1, U1.8 (PH)
- new net: C13.2, U3.6 (UCAP)
- new net: C9.2, U3.16 (XTAL2), Y1.1
- new net: C8.2, U3.17 (XTAL1), Y1.4
- new net: LED1.1 (A), R2.2
- new net: J3.A5 (CC1), R16.1
- new net: J3.B5 (CC2), R15.1
- new net: C1.2, U1.1 (BOOT)
- new net +1V8: C15.2, C16.1, C17.1, C19.1, R17.1, R18.1, R19.1, R20.1, TP11.1, U4.2 (Vout), U5.1 (V_{CCA}), U5.8 (OE), U6.1 (AVDDVCSEL), U6.11 (AVDD)
- new net +24V: C2.1, DC1.4, TP1.1, U1.5 (EN), U1.7 (VIN), U7.1 (IP+), U7.2 (IP+)
- new net +5V: C10.2, C11.2, C14.2, C18.1, C20.2, C4.1, C6.2, C7.2, FPC_MB1.6, J2.2 (Pin_2), JP1.1 (A), L1.2, R3.1, R5.1, R6.1, R7.1, TP10.1, U2.16 (VDD), U3.14 (VCC), U3.2 (UVCC), U3.24 (AVCC), U3.34 (VCC), U3.44 (AVCC), U4.3 (Vin), U5.14 (V_{CCB}), U7.8 (VCC)
- new net +5VA: FPC_HMI1.6, J1.1 (Pin_1), SW1.2, SW2.2, SW3.2, SW4.2, SW5.2
- new net CS_HMIside: FPC_HMI1.11, J1.6 (Pin_6), TP5.1
- new net CS_MBside: FPC_MB1.11, U3.8 (PB0)
- new net D+: R8.2, U3.4 (D+)
- new net D-: R9.2, U3.3 (D-)
- new net DC_HMIside: FPC_HMI1.10, J1.5 (Pin_5), TP4.1
- new net DC_MBside: FPC_MB1.10, U3.28 (PB4)
- new net GND: C10.1, C11.1, C12.1, C13.1, C14.1, C15.1, C16.2, C17.2, C18.2, C19.2, C2.2, C20.1, C21.1, C22.1, C4.2, C6.1, C7.1, C8.1, C9.1, D1.2 (A), DC1.2, DC1.3, FPC_MB1.13, FPC_MB1.14, FPC_MB1.7, H1.1, H2.1, J2.6 (Pin_6), J3.A1_B12 (GND), J3.B1_A12 (GND), J3.SH1 (SHELL_GND), J3.SH2 (SHELL_GND), J3.SH3 (SHELL_GND), J3.SH4 (SHELL_GND), J4.2, J5.3, LED1.2 (K), R10.2, R11.2, R12.2, R13.2, R14.2, R15.2, R16.2, R4.2, RST1.1, TP9.1, U1.6 (GND), U1.9 (GNDPAD), U2.1 (A0), U2.2 (A1), U2.3 (A2), U2.8 (GND), U3.15 (GND), U3.23 (GND), U3.33 (~{HWB}/PE2), U3.35 (GND), U3.43 (GND), U3.5 (UGND), U4.1 (GND), U5.7 (GND), U6.12 (GND4), U6.2 (AVSSVCSEL), U6.3 (GND), U6.4 (GND2), U6.6 (GND3), U7.5 (GND), Y1.2 (G), Y1.3 (G)
- new net GNDA: FPC_HMI1.13, FPC_HMI1.14, FPC_HMI1.7, J1.2 (Pin_2)
- new net GPIO1_VL53: TP14.1, U3.20 (PD2), U5.11 (B3)
- new net HMI_~{INT}: TP8.1, U2.13 (~{INT}), U3.21 (PD3)
- new net Imotor: C22.2, R21.2, TP19.1, U3.41 (PF0)
- new net MISO: J2.1 (Pin_1), U3.11 (PB3)
- new net MOSI: FPC_MB1.9, J2.4 (Pin_4), U3.10 (PB2)
- new net MOSI_HMIside: FPC_HMI1.9, J1.4 (Pin_4), TP3.1
- new net Mdir: J5.1, U3.31 (PC6)
- new net Mpwm: J5.2, U3.30 (PB6)
- new net RESET: J2.5 (Pin_5), R5.2, RST1.2, TP7.1, U3.13 (~{RESET})
- new net RST_HMIside: FPC_HMI1.12, J1.7 (Pin_7), TP6.1
- new net RST_MBside: FPC_MB1.12, U3.29 (PB5)
- new net SCK: FPC_MB1.8, J2.3 (Pin_3), U3.9 (PB1)
- new net SCK_HMIside: FPC_HMI1.8, J1.3 (Pin_3), TP2.1
- new net SCL: R6.2, TP12.1, U2.14 (SCL), U3.18 (PD0), U5.13 (B1)
- new net SDA: R7.2, TP13.1, U2.15 (SDA), U3.19 (PD1), U5.12 (B2)
- new net SW1_HMIside: FPC_HMI1.1, SW1.1
- new net SW1_MBside: FPC_MB1.1, R10.1, U2.4 (P0)
- new net SW2_HMIside: FPC_HMI1.2, SW2.1
- new net SW2_MBside: FPC_MB1.2, R11.1, U2.5 (P1)
- new net SW3_HMIside: FPC_HMI1.3, SW3.1
- new net SW3_MBside: FPC_MB1.3, R12.1, U2.6 (P2)
- new net SW4_HMIside: FPC_HMI1.4, SW4.1
- new net SW4_MBside: FPC_MB1.4, R13.1, U2.7 (P3)
- new net SW5_HMIside: FPC_HMI1.5, SW5.1
- new net SW5_MBside: FPC_MB1.5, R14.1, U2.9 (P4)
- new net VBUS: J3.A4_B9 (VBUS), J3.B4_A9 (VBUS), U3.7 (VBUS)
- no-connect marks 0 -> 20
Other:
- removed sheet Motor-driver
- removed sheet laser-meter
- note added: "Addr: 0x20"
- note added: "C53207173"
- note added: "IO expander HMI switch"
- note added: "LCD screen connection"
- note added: "Motherboard to HMI connection"
- note added: "Motor current sensing and command"
- note added: "Optical height monitor"
- note added: "Vout = 2.5 + I x 0.4 V"
- note added: "addr: 0x52"
- note added: "max voltage: 1.8 V"

Commit message: finish pcb
Parts:
- U4: value XC6206P182MR -> XC6206P282MR
Connections:
- net +1V8 renamed +2V8
Other:
- note added: "max voltage: 2.8 V"
- note removed: "max voltage: 1.8 V"
