File: hardware/desktopia.kicad_sch (KiCad schematic)
At the start: 88 parts, among them J1 LCD_Connector, J2 Prog_Connector, J3 USB4105GFA, J4 PowerMotor, J5 MotorCommandCon, SW1 SW_Push, SW2 SW_Push, SW3 SW_Push, SW4 SW_Push, SW5 SW_Push, U1 TPS5430DDA, U2 TCA9554DB, U3 ATmega32U4-A, U4 XC6206P282MR, U5 TXS0104EPW, U6 VL53L1CBV0FY_1, U7 CC6905S8-5FB005, Y1 X322516MLB4SI

Commit message: HMI board with its own RP2040, linked to the motherboard by RS-485 over an RJ11 cord
- motherboard firmware: HMI link master (Serial1 + DE on PD4), TCA9554 and screen driver removed,
  Up+Down stop of a preset move, motor stopped when the link is lost
- hmi_firmware: RP2040 (arduino-pico), link slave with A/B polarity detection, screen on core 1
- shared/hmi_link: frame protocol (CRC-16) and screen model used by both firmwares
- simulation of both boards over a simulated RS-485 bus (628 checks)
- schematics: RJ11 + THVD1450 on the motherboard, new desktopia_HMI.kicad_sch

Co-Authored-By: Claude Opus 5.5 <noreply@anthropic.com>
Parts:
- removed C10: 100nF, Capacitor_SMD:C_0402_1005Metric, symbol Device:C_Small
- removed C11: 1uF, Capacitor_SMD:C_0402_1005Metric, symbol Device:C_Small
- removed FPC_HMI1, FPC_MB1: F2D12U-A1G1-ER, JLCImport:F2D12U-A1G1-ER, symbol JLCImport:F2D12U-A1G1-ER
- removed J1: LCD_Connector, JLCImport:LCD_round_screen, symbol Connector:Conn_01x07_Pin
- removed R10, R11, R12, R13, R14: 10k, Resistor_SMD:R_0402_1005Metric, symbol Device:R
- removed SW1, SW2, SW3, SW4, SW5: SW_Push, JLCImport:PG1350, symbol Switch:SW_Push
- removed TP2, TP3, TP4, TP5, TP6, TP8: TestPoint, TestPoint:TestPoint_Pad_D1.0mm, symbol Connector:TestPoint
- removed U2: TCA9554DB, Package_SO:SSOP-16_5.3x6.2mm_P0.65mm, symbol Interface_Expansion:TCA9554DB
- added C23: 100nF, Capacitor_SMD:C_0402_1005Metric, symbol Device:C_Small
- added C24: 10uF, Capacitor_SMD:C_0603_1608Metric, symbol Device:C_Small
- added F1: PTC 500mA, Fuse:Fuse_1206_3216Metric, symbol Device:Polyfuse_Small
- added J6: RJ11 6P6C, Connector_RJ:RJ12_Amphenol_54601-x06_Horizontal, symbol Connector:RJ12
- added R22, R23: 4.7k, Resistor_SMD:R_0402_1005Metric, symbol Device:R
- added R24: 120, Resistor_SMD:R_0402_1005Metric, symbol Device:R
- added U8: THVD1450D, Package_SO:SOIC-8_3.9x4.9mm_P1.27mm, symbol Interface_UART:THVD1450D
Connections:
- net +5V: now also C23.1, F1.1, R22.1, U8.8 (VCC)
- net GND: now also C23.2, C24.2, J6.2, J6.5, R23.2, U8.5 (GND)
- net GPIO1_VL53: no longer U3.20 (PD2)
- net RS485_DE: now reaches U3.25 (PD4)
- net RS485_DE: now also U8.2 (~{RE}), U8.3 (DE)
- net CS_MBside: no longer names the net of U3.8 (PB0)
- net DC_MBside: no longer names the net of U3.28 (PB4)
- net HMI_~{INT} renamed RS485_DI
- net RS485_DI: now also U8.4 (DI)
- net RST_MBside: no longer names the net of U3.29 (PB5)
- new net +5V_HMI: C24.1, F1.2, J6.1, J6.6
- new net RS485_A: J6.3, R22.2, R24.1, U8.6 (A)
- new net RS485_B: J6.4, R23.1, R24.2, U8.7 (B)
- new net RS485_RO: U3.20 (PD2), U8.1 (RO)
- no-connect marks 20 -> 19
Other:
- note added: "I2C pull-ups"
- note added: "J6 pin-out (6P6C, straight or reversed cord): 1 = +5V 2 = GND 3 = A 4 = B 5 = GND 6 = +5V A reversed cord only swaps A and B: the HMI board detects it. Never plug J6 into a telephone wall socket."
- note added: "Motherboard to HMI board link: RS-485 over an RJ11 cord"
- note added: "R22 / R23: bias. R24 (DNP): 120R termination, only for cords over ~5 m (then R22 / R23 = 680R)."
- note removed: "Addr: 0x20"
- note removed: "C53207173"
- note removed: "IO expander HMI switch"
- note removed: "LCD screen connection"
- note removed: "Motherboard to HMI connection"
- moved on the sheet: R6, R7
