File: hardware/desktopia/desktopia.kicad_sch (KiCad schematic)
At the start: 74 parts, among them J2 Prog_Connector, J3 USB4105GFA, J4 PowerMotor, J5 MotorCommandCon, J6 RJ11 6P6C, U1 TPS5430DDA, U3 ATmega32U4-A, U4 XC6206P282MR, U5 TXS0104EPW, U6 VL53L1CBV0FY_1, U7 CC6905S8-5FB005, U8 THVD1450D, Y1 X322516MLB4SI

Commit message: hardware: JLCPCB part numbers, safe TPS5430 enable, 24 V screw terminal, INA226 current sensor
- Every assembled part gets LCSC / jlcpcb PartNumber fields, Basic parts first (SP485EEN, SP3485EN,
  W25Q128JV, 12 MHz crystal with 33 pF, TS-1088 buttons, ...).
- TPS5430 ENA was tied to the 24 V input (7 V absolute maximum) and burnt the regulator: left open now.
- C25 10 uF 50 V ceramic input capacitor next to C2.
- 1.5 A barrel jack DC1 replaced by the 5.08 mm screw terminal J7.
- Analog CC6905 replaced by a 2 mOhm shunt + INA226 on I2C (0x40), alert on PE6; PF0 is free.

Co-Authored-By: Claude Opus 5.5 <noreply@anthropic.com>
Parts:
- removed C21: 1nF, Capacitor_SMD:C_0402_1005Metric, symbol Device:C_Small
- removed C22: 100pF, Capacitor_SMD:C_0402_1005Metric, symbol Device:C_Small
- removed DC1: DC050-2_5-T, JLCImport:DC050-2_5-T, symbol JLCImport:DC050-2_5-T
- removed R21: 100, Resistor_SMD:R_0402_1005Metric, symbol Device:R
- removed TP19: TestPoint, TestPoint:TestPoint_Pad_D1.0mm, symbol Connector:TestPoint
- removed U7: CC6905S8-5FB005, Package_SO:SOP-8_3.76x4.96mm_P1.27mm, symbol JLCImport:CC6905S8-5FB005
- added C25: 10uF, Capacitor_SMD:C_1206_3216Metric, symbol Device:C_Small
- added J7: Power24V, JLCImport:C508128L-2P0G36, symbol JLCImport:C508128L-2P0G36
- added R25: 2mR 3W, Resistor_SMD:R_2512_6332Metric, symbol Device:R
- added R26: 10k, Resistor_SMD:R_0402_1005Metric, symbol Device:R
- added U9: INA226AIDGSR, Package_SO:TSSOP-10_3x3mm_P0.5mm, symbol Sensor_Energy:INA226
- C1: LCSC (none) -> C15195
- C12, C17, C18, C19, C20, C23, C6, C7: LCSC (none) -> C1525
- C13, C14, C15: LCSC (none) -> C52923
- C16: LCSC (none) -> C23733
- C2: jlcpcb PartNumber (none) -> C18221489
- C24: LCSC (none) -> C19702; jlcpcb PartNumber (none) -> C19702
- C4: LCSC C249510 -> C72507; Manufacturer Lelon -> ROQANG; Manufacturer Part VE-330M1ATR-0505 -> RVT1E330M0505; jlcpcb PartNumber (none) -> C72507
- C8, C9: LCSC (none) -> C32949
- D1: LCSC (none) -> C2480
- F1: LCSC (none) -> C70075; jlcpcb PartNumber (none) -> C70075
- J3: LCSC (none) -> C3020560; jlcpcb PartNumber (none) -> C3020560
- J4: jlcpcb PartNumber (none) -> C49291865
- J5: jlcpcb PartNumber (none) -> C49023012
- J6: LCSC (none) -> C3097716; jlcpcb PartNumber (none) -> C3097716
- L1: value 84uH -> 85uH; LCSC (none) -> C5374269
- LED1: jlcpcb PartNumber (none) -> C2286
- R1, R2: LCSC (none) -> C25076
- R15, R16: LCSC (none) -> C25905
- R17, R18, R4, R6, R7: LCSC (none) -> C25890
- R19, R20, R3, R5: LCSC (none) -> C25744
- R22, R23: LCSC (none) -> C25900; jlcpcb PartNumber (none) -> C25900
- R24: LCSC (none) -> C25079; jlcpcb PartNumber (none) -> C25079
- R8, R9: LCSC (none) -> C25092
- RST1: value SW_Push -> TS-1088-AR02016; footprint JLCImport:DTS41 -> Button_Switch_SMD:SW_SPST_TS-1088-xR020; LCSC (none) -> C720477; jlcpcb PartNumber (none) -> C720477
- U1: LCSC (none) -> C9864
- U3: LCSC (none) -> C44854; jlcpcb PartNumber (none) -> C44854
- U4: LCSC C51886219 -> C347374; Manufacturer TECH PUBLIC -> UMW(Youtai Semiconductor Co., Ltd.); Manufacturer Part XC6206P182MR -> XC6206P282MR; jlcpcb PartNumber (none) -> C347374
- U5: LCSC (none) -> C44955
- U6: jlcpcb PartNumber (none) -> C2970716
- U8: value THVD1450D -> SP485EEN-L/TR; symbol Interface_UART:THVD1450D -> Interface_UART:MAX485E; LCSC (none) -> C6855; jlcpcb PartNumber (none) -> C6855
- Y1: LCSC (none) -> C13738
Connections:
- net +24V: now also C25.1, J7.1, R25.1, U9.10 (Vin+); no longer U1.5 (EN)
- net +5V: now also C20.1, R26.1, U9.6 (VS); no longer C20.2
- net GND: now also C20.2, C25.2, J7.2, U9.1 (A1), U9.2 (A0), U9.7 (GND); no longer C20.1
- net SCL: now also U9.5 (SCL)
- net SDA: now also U9.4 (SDA)
- net MOTOR_24V: now reaches J4.1
- net MOTOR_24V: now also R25.2, U9.8 (Vbus), U9.9 (Vin-)
- net I_ALERT: now reaches U3.1 (PE6)
- net I_ALERT: now also R26.2, U9.3 (~{Alert})
- net Imotor: no longer names the net of U3.41 (PF0)
- no-connect marks 19 -> 20
Other:
- note added: "24 V supply input, 18 A screw terminal (it carries the motor current)"
- note added: "ENA left open: internal 1.5 MOhm pull-up, 7 V absolute maximum. Never tie it to VIN (24 V destroys the TPS5430)."
- note added: "INA226: I2C address 0x40 (A0 = A1 = GND), alert on PE6. R25 2 mOhm: +-41 A full scale, 1.25 mA resolution, 0.34 W at 13 A. Kelvin-connect Vin+ / Vin- right at the R25 pads. +24V / MOTOR_24V: copper for 15 A (pours, or >= 5 mm in 1 oz)."
- note removed: "Vout = 2.5 + I x 0.4 V"

Commit message: hardware: JLCPCB cost pass, motor input with margin, BSS138 level shifters
Motherboard:
- Extended part numbers 12 -> 9: TXS0104E -> BSS138 level shifters (Preferred),
  C4 electrolytic -> 2 x 47 uF ceramic with the TI SLVA237 compensation,
  J5 -> the same KF128 terminal as J4 / J7, J3 GCT USB4105 (out of stock)
  -> G-Switch GT-USB-7010ASV, R1 + R2 -> R1, F1 -> 30 V PTC.
- 24 V input with margin: SMBJ28A TVS, 220 uF 50 V bulk, 24 A terminals.
  5 V rail good for 1.5 A: 22 uH 1.8 A inductor, SS34.
- Sensor rail stays at 2.8 V (VL53L1CB typical, 0.7 V under its maximum).
  VL53L1CB GPIO1 -> TOF_INT on PB4 (PCINT4) through a third BSS138.
- 10k pull-downs on Mpwm / Mdir. INA226 alert kept on INT6, with a 4.7k
  pull-up and a 100 pF filter.

HMI: USB-C G-Switch GT-USB-7010ASV ($0.09 instead of $0.19).

READMEs and the firmware pin comments follow the schematics.

Co-Authored-By: Claude Opus 5.5 <noreply@anthropic.com>
Parts:
- removed C18, C19: 100nF, Capacitor_SMD:C_0402_1005Metric, symbol Device:C_Small
- removed R2: 100, Resistor_SMD:R_0402_1005Metric, symbol Device:R
- removed TP14: TestPoint, TestPoint:TestPoint_Pad_D1.0mm, symbol Connector:TestPoint
- removed U5: TXS0104EPW, Package_SO:TSSOP-14_4.4x5mm_P0.65mm, symbol Logic_LevelTranslator:TXS0104EPW
- added C26: 47uF, Capacitor_SMD:C_1206_3216Metric, symbol Device:C_Small
- added C27: 2.2nF, Capacitor_SMD:C_0603_1608Metric, symbol Device:C_Small
- added C28: 100nF, Capacitor_SMD:C_0402_1005Metric, symbol Device:C_Small
- added C29, C30: 100pF, Capacitor_SMD:C_0402_1005Metric, symbol Device:C_Small
- added D2: SMBJ28A, Diode_SMD:D_SMB, symbol Diode:SM6T33A
- added Q1, Q2, Q3: BSS138, Package_TO_SOT_SMD:SOT-23, symbol Transistor_FET:BSS138
- added R27: 470, Resistor_SMD:R_0402_1005Metric, symbol Device:R
- added R28, R29, R30: 10k, Resistor_SMD:R_0402_1005Metric, symbol Device:R
- C2: value 4.7uF -> 220uF; footprint JLCImport:RVT1H4R7M0405_C18221489 -> Capacitor_SMD:CP_Elec_10x10; symbol JLCImport:RVT1H4R7M0405_C18221489 -> Device:C_Polarized; LCSC C18221489 -> C2887271; Manufacturer RS -> KNSCHA; Manufacturer Part RVT1H4R7M0405 -> RVT220UF50V67RV0021; Voltage (none) -> 50V; jlcpcb PartNumber C18221489 -> C2887271
- C4: value 33uF -> 47uF; footprint JLCImport:VE-330M1A0505-TRO -> Capacitor_SMD:C_1206_3216Metric; symbol JLCImport:VE-330M1A0505-TRO -> Device:C_Small; LCSC C72507 -> C96123; Manufacturer ROQANG -> Samsung Electro-Mechanics; Manufacturer Part RVT1E330M0505 -> CL31A476MPHNNNE; Voltage (none) -> 10V X5R; jlcpcb PartNumber C72507 -> C96123
- D1: value SS14 -> SS34; symbol Diode:SS14 -> Diode:SS34; LCSC C2480 -> C8678; jlcpcb PartNumber C2480 -> C8678
- F1: LCSC C70075 -> C720075; jlcpcb PartNumber C70075 -> C720075
- J3: value USB4105GFA -> GT-USB-7010ASV; footprint JLCImport:GCT_USB4105GFA -> Connector_USB:USB_C_Receptacle_G-Switch_GT-USB-7010ASV; symbol USB4105GFA:USB4105GFA -> Connector:USB_C_Receptacle_USB2.0_16P; Availability In Stock -> (none); Check_prices https://www.snapeda.com/parts/USB4105GFA/Global+Connector+T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 -> (none); LCSC C3020560 -> C2988369; MANUFACTURER Global Connector Technology -> (none); MAXIMUM_PACKAGE_HEIGHT 3.31mm -> (none); MF Global Connector Technology -> (none); MP USB4105GFA -> (none); Manufacturer (none) -> G-Switch; Manufacturer Part (none) -> GT-USB-7010ASV; PARTREV B3 -> (none); Package None -> (none); Price None -> (none); Purchase-URL https://www.snapeda.com/api/url_track_click_mouser/?unipart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 -> (none); STANDARD Manufacturer Recommendations -> (none); SnapEDA_Link https://www.snapeda.com/parts/USB4105GFA/Global+Connector+T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 -> (none); jlcpcb PartNumber C3020560 -> C2988369; now in the parts list
- J4, J7: LCSC C49291865 -> C474952; Manufacturer JXTCONN -> Cixi Kefa Elec; Manufacturer Part C508128L-2P0G36 -> KF128-5.08-2P-AA; jlcpcb PartNumber C49291865 -> C474952
- J5: footprint JLCImport:ZX-DG28L-2_54-3P -> JLCImport:C508128L-2P0G36; symbol JLCImport:ZX-DG28L-2_54-3P -> JLCImport:C508128L-2P0G36; LCSC C49023012 -> C474952; Manufacturer Megastar -> Cixi Kefa Elec; Manufacturer Part ZX-DG28L-2.54-3P -> KF128-5.08-2P-AA; jlcpcb PartNumber C49023012 -> C474952
- L1: value 85uH -> 22uH; footprint JLCImport:L5.8 -> Inductor_SMD:L_Sunlord_SWPA6045S; LCSC C5374269 -> C83454; Manufacturer (none) -> Sunlord; Manufacturer Part (none) -> SWPA6045S220MT; jlcpcb PartNumber C5374269 -> C83454
- R1: value 100 -> 470; LCSC C25076 -> C25117; jlcpcb PartNumber C25076 -> C25117
- R26: value 10k -> 4.7k; LCSC C25744 -> C25900; jlcpcb PartNumber C25744 -> C25900
Connections:
- net +24V: now also D2.1 (A1)
- net +2V8: now also Q1.1 (G), Q2.1 (G), Q3.1 (G)
- net +5V: now also C26.1, C27.1, R30.1
- net GND: now also J3.A1 (GND), J3.A12 (GND), J3.B1 (GND), J3.B12 (GND), J3.SH (SHIELD), C26.2, C28.2, C29.2, C30.2, D2.2 (A2), R28.2, R29.2; no longer J3.A1_B12 (GND), J3.B1_A12 (GND), J3.SH1 (SHELL_GND), J3.SH2 (SHELL_GND), J3.SH3 (SHELL_GND), J3.SH4 (SHELL_GND), J5.3
- net I_ALERT: now also C30.1
- net Mdir: now also R29.1
- net Mpwm: now also R28.1
- net SCL: now also Q1.3 (D)
- net SDA: now also Q2.3 (D)
- net VBUS: now also J3.A4 (VBUS), J3.A9 (VBUS), J3.B4 (VBUS), J3.B9 (VBUS); no longer J3.A4_B9 (VBUS), J3.B4_A9 (VBUS)
- net SCL_2V8: now reaches R17.2, TP15.1, U6.10 (SCL)
- net SCL_2V8: now also Q1.2 (S)
- net at R3.2, R4.1, U1.4 (VSENSE): now also C27.2, C29.1, R27.1
- net SDA_2V8: now reaches R18.2, TP16.1, U6.9 (SDA)
- net SDA_2V8: now also Q2.2 (S)
- net TOF_INT_2V8: now reaches R20.2, TP17.1, U6.7 (GPIO1)
- net TOF_INT_2V8: now also Q3.2 (S)
- net at R1.2: now also LED1.1 (A)
- net USB_D+: now reaches J3.A6 (D+), J3.B6 (D+), R8.1
- net USB_D-: now reaches J3.A7 (D-), J3.B7 (D-), R9.1
- net USB_CC1: now reaches J3.A5 (CC1), R16.1
- net USB_CC2: now reaches J3.B5 (CC2), R15.1
- net TOF_INT: now reaches U3.28 (PB4)
- net TOF_INT: now also Q3.3 (D), R30.2
- new net: C28.1, R27.2
- no-connect marks 20 -> 17
Other:
- note added: "24 V supply input, 24 A screw terminal (it carries the motor current)"
- note added: "AVDD 2.8 V (2.6 - 3.5 V)"
- note added: "Ceramic output compensation (TI SLVA237): L1 22 uH, C4 + C26 2 x 47 uF: f_LC ~ 4.7 kHz. C27 / R27 / C28 / C29: crossover 14-27 kHz, phase margin > 60 deg, 0.1 to 1.5 A."
- note added: "D2 clamps motor and hot-plug spikes below the 40 V absolute maximum of U1 and U9. C2: 24 V bulk."
- note added: "J5: DIR + PWM only. Logic GND via J4 pin 2."
- note added: "Motor pull-downs"
- note added: "Q1 / Q2 / Q3 (BSS138, Vgs(th) <= 1.5 V) replace the TXS0104E. 5 V side: SCL, SDA, TOF_INT (PB4 / PCINT4). Sensor side: SCL_2V8, SDA_2V8, TOF_INT_2V8 (GPIO1). A low from the MCU stays under the 0.6 V VIL of the sensor."
- note added: "ToF INT pull-up"
- note removed: "24 V supply input, 18 A screw terminal (it carries the motor current)"
- note removed: "max voltage: 2.8 V"

Commit message: hardware: motor supply switch, schematics redrawn with fewer labels, re-annotation
Motherboard:
- Q5 P-MOSFET high-side switch on the driver supply (Q4 gate driver, D3 clamp,
  C21 soft start, R22 pull-down), driven by PD7 (MOTOR_PWR); TP13 on MOTOR_SW
- Schematic redrawn: wires instead of labels inside each block (76 -> 22 labels),
  same netlist
- J6 motor command terminal: 3 pins again (ZX-DG28L-2.54-3P), pin 3 = driver logic GND
- C6 24 V bulk: 220 uF 10 x 10 mm -> 100 uF 8 x 10 mm (C970687), same cable damping
- Re-annotated; TP9 on TOF_INT, H3 mounting hole, J3 and Y1 symbols updated,
  HWB left open; notes and README follow the new references

HMI board:
- Schematic redrawn without labels (70 -> 0), same netlist

The PCB files are not part of this commit.

Co-Authored-By: Claude Opus 5.5 <noreply@anthropic.com>
Parts:
- removed R16: 5.1k, Resistor_SMD:R_0402_1005Metric, symbol Device:R
- added C21: 100nF, Capacitor_SMD:C_0402_1005Metric, symbol Device:C_Small
- added D3: BZT52C15, Diode_SMD:D_SOD-123, symbol Device:D_Zener
- added D4: SS34, Diode_SMD:D_SMA, symbol Diode:SS34
- added H3: MountingHole_Pad, MountingHole:MountingHole_2.2mm_M2_Pad, symbol Mechanical:MountingHole_Pad
- added Q4: BSS138, Package_TO_SOT_SMD:SOT-23, symbol Transistor_FET:BSS138
- added Q5: IPD90P04P4-05, Package_TO_SOT_SMD:TO-252-2, symbol Transistor_FET:Q_PMOS_GDS
- added R19: 5.1k, Resistor_SMD:R_0402_1005Metric, symbol Device:R
- added R20, R21: 100k, Resistor_SMD:R_0402_1005Metric, symbol Device:R
- added R22: 10k, Resistor_SMD:R_0402_1005Metric, symbol Device:R
- added TP13, TP9: TestPoint, TestPoint:TestPoint_Pad_D1.0mm, symbol Connector:TestPoint
- C6: renamed from C2; value 220uF -> 100uF; footprint Capacitor_SMD:CP_Elec_10x10 -> Capacitor_SMD:CP_Elec_8x10; LCSC C2887271 -> C970687; Manufacturer KNSCHA -> DMBJ; Manufacturer Part RVT220UF50V67RV0021 -> RVT1H101M0810; jlcpcb PartNumber C2887271 -> C970687
- J6: renamed from J5; footprint JLCImport:C508128L-2P0G36 -> JLCImport:ZX-DG28L-2_54-3P; symbol JLCImport:C508128L-2P0G36 -> JLCImport:ZX-DG28L-2_54-3P; LCSC C474952 -> C49023012; Manufacturer Cixi Kefa Elec -> Megastar; Manufacturer Part KF128-5.08-2P-AA -> ZX-DG28L-2.54-3P; jlcpcb PartNumber C474952 -> C49023012
- Y1: symbol Device:Crystal_GND23_Small -> Device:Crystal_GND24_Small
- renumbered C14 to C1, C17 to C10, C29 to C11, C28 to C12, C6 to C13, C7 to C14, C8 to C15, C9 to C16, C12 to C17, C23 to C18, C13 to C19, C15 to C2, C24 to C20, C20 to C22, C30 to C23, C1 to C3, C27 to C4, C25 to C5, C4 to C7, C26 to C8, C16 to C9, J7 to J1, J6 to J4, J4 to J5, R6 to R1, R30 to R10, R20 to R11, R5 to R12, R8 to R13, R22 to R14, R9 to R15, R24 to R16, R23 to R17, R15 to R18, R17 to R2, R25 to R23, R29 to R24, R26 to R25, R28 to R26, R1 to R3, R3 to R4, R7 to R5, R18 to R6, R4 to R7, R19 to R8, R27 to R9, TP10 to TP1, TP17 to TP10, TP7 to TP11, TP9 to TP12, TP11 to TP2, TP12 to TP3, TP15 to TP4, TP1 to TP5, TP13 to TP6, TP16 to TP7, TP18 to TP8, U4 to U1, U1 to U2, U6 to U3, U3 to U4, U8 to U5, U9 to U6
Connections:
- net GND: now also J6.3, Y1.4 (G), D4.2 (A), H3.1, Q4.2 (S), R19.2, R22.2; no longer U4.33 (~{HWB}/PE2), Y1.3 (G)
- net MOTOR_24V: now also D3.1 (K), Q5.3 (S), R21.2; no longer J5.1
- net TOF_INT: now also TP9.1
- net at C15.2, U4.17 (XTAL1): now also Y1.3; no longer Y1.4
- net MOTOR_PWR: now reaches U4.27 (PD7)
- net MOTOR_PWR: now also Q4.1 (G), R22.1
- net D+: no longer names the net of R13.2, U4.4 (D+)
- net D-: no longer names the net of R15.2, U4.3 (D-)
- net MISO: no longer names the net of J2.1 (Pin_1), U4.11 (PB3)
- net MOSI: no longer names the net of J2.4 (Pin_4), U4.10 (PB2)
- net RS485_A: no longer names the net of J4.3, R14.2, R16.1, U5.6 (A)
- net RS485_B: no longer names the net of J4.4, R16.2, R17.1, U5.7 (B)
- net RS485_DE: no longer names the net of U4.25 (PD4), U5.2 (~{RE}), U5.3 (DE)
- net RS485_DI: no longer names the net of U4.21 (PD3), U5.4 (DI)
- net RS485_RO: no longer names the net of U4.20 (PD2), U5.1 (RO)
- net SCK: no longer names the net of J2.3 (Pin_3), U4.9 (PB1)
- net SCL_2V8: no longer names the net of Q1.2 (S), R2.2, TP4.1, U3.10 (SCL)
- net SDA_2V8: no longer names the net of Q2.2 (S), R6.2, TP7.1, U3.9 (SDA)
- net TOF_INT_2V8: no longer names the net of Q3.2 (S), R11.2, TP10.1, U3.7 (GPIO1)
- net USB_CC1: no longer names the net of J3.A5 (CC1)
- net USB_CC1: now also R19.1
- net USB_CC2: no longer names the net of J3.B5 (CC2), R18.1
- net USB_D+: no longer names the net of J3.A6 (D+), J3.B6 (D+), R13.1
- net USB_D-: no longer names the net of J3.A7 (D-), J3.B7 (D-), R15.1
- net VBUS: no longer names the net of J3.A4 (VBUS), J3.A9 (VBUS), J3.B4 (VBUS), J3.B9 (VBUS), U4.7 (VBUS)
- new net: C21.1, D3.2 (A), Q5.1 (G), R20.1, R21.1
- new net: Q4.3 (D), R20.2
- new net MOTOR_SW: C21.2, D4.1 (K), J5.1, Q5.2 (D), TP13.1
- no-connect marks 17 -> 15
Other:
- note added: "Ceramic output compensation (TI SLVA237): L1 22 uH, C7 + C8 2 x 47 uF: f_LC ~ 4.7 kHz. C4 / R9 / C12 / C11: crossover 14-27 kHz, phase margin > 60 deg, 0.1 to 1.5 A."
- note added: "D2 clamps motor and hot-plug spikes below the 40 V absolute maximum of U2 and U6. C6: 24 V bulk."
- note added: "ENA left open: internal 1.5 MOhm pull-up"
- note added: "INA226: I2C address 0x40 (A0 = A1 = GND), alert on PE6. R23 2 mOhm: +-41 A full scale, 1.25 mA resolution, 0.34 W at 13 A. Kelvin-connect Vin+ / Vin- right at the R23 pads. +24V / MOTOR_24V / MOTOR_SW: copper for 15 A (pours, or >= 5 mm in 1 oz)."
- note added: "J4 pin-out (6P6C, straight or reversed cord): 1 = +5V 2 = GND 3 = A 4 = B 5 = GND 6 = +5V A reversed cord only swaps A and B: the HMI board detects it. Never plug J4 into a telephone wall socket."
- note added: "J6: DIR, PWM and logic GND to the MD10C input header."
- note added: "Link to the HMI board: RS-485 over an RJ11 cord"
- note added: "MOTOR_PWR high: Q5 on (Vgs -12 V). R22 keeps it off in reset. C21 / R20: ~15 ms soft start. Cut only with the PWM at 0."
- note added: "Motor supply: shunt + INA226, switch, driver connectors"
- note added: "Mounting holes"
- note added: "Q1 / Q2 / Q3 (BSS138, Vgs(th) <= 1.5 V) replace the TXS0104E. 5 V side: SCL, SDA, TOF_INT (PB4 / PCINT4). Sensor side (2.8 V): SCL, SDA and GPIO1 of U3. A low from the MCU stays under the 0.6 V VIL of the sensor."
- note added: "R14 / R17: bias. R16 (DNP): 120R termination, only for cords over ~5 m (then R14 / R17 = 680R)."
- note removed: "Ceramic output compensation (TI SLVA237): L1 22 uH, C4 + C26 2 x 47 uF: f_LC ~ 4.7 kHz. C27 / R27 / C28 / C29: crossover 14-27 kHz, phase margin > 60 deg, 0.1 to 1.5 A."
- note removed: "D2 clamps motor and hot-plug spikes below the 40 V absolute maximum of U1 and U9. C2: 24 V bulk."
- note removed: "ENA left open: internal 1.5 MOhm pull-up, 7 V absolute maximum. Never tie it to VIN (24 V destroys the TPS5430)."
- note removed: "I2C pull-ups"
- note removed: "INA226: I2C address 0x40 (A0 = A1 = GND), alert on PE6. R25 2 mOhm: +-41 A full scale, 1.25 mA resolution, 0.34 W at 13 A. Kelvin-connect Vin+ / Vin- right at the R25 pads. +24V / MOTOR_24V: copper for 15 A (pours, or >= 5 mm in 1 oz)."
- note removed: "J5: DIR + PWM only. Logic GND via J4 pin 2."
- note removed: "J6 pin-out (6P6C, straight or reversed cord): 1 = +5V 2 = GND 3 = A 4 = B 5 = GND 6 = +5V A reversed cord only swaps A and B: the HMI board detects it. Never plug J6 into a telephone wall socket."
- note removed: "Motherboard to HMI board link: RS-485 over an RJ11 cord"
- note removed: "Motor current sensing and command"
- note removed: "Motor pull-downs"
- note removed: "Q1 / Q2 / Q3 (BSS138, Vgs(th) <= 1.5 V) replace the TXS0104E. 5 V side: SCL, SDA, TOF_INT (PB4 / PCINT4). Sensor side: SCL_2V8, SDA_2V8, TOF_INT_2V8 (GPIO1). A low from the MCU stays under the 0.6 V VIL of the sensor."
- note removed: "R22 / R23: bias. R24 (DNP): 120R termination, only for cords over ~5 m (then R22 / R23 = 680R)."
- note removed: "ToF INT pull-up"
- moved on the sheet: C1, C10, C17, C18, C19, C2, C20, C22, C23, C9, F1, H1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
